Commit message: modified the sensors and main xacro files changing the weight of the jetank and the camera remapping

File: jetank_description/urdf/jetank_main.xacro (robot description, xacro)
@@ -53,5 +53,5 @@
     <xacro:property name="BEARING_material"                 value="0.67 0.74 0.67 1" />
     <!-- mass -->
-    <xacro:property name="base_link_mass"               value="0.7639308708503839" />
+    <xacro:property name="base_link_mass"               value="2.7639308708503839" />
     <xacro:property name="DRIVER_WHEEL_L_mass"          value="0.1049698213829899" />
     <xacro:property name="DRIVER_WHEEL_R_mass"          value="0.1049698213829899" />

File: jetank_description/urdf/jetank_sensors.xacro (robot description, xacro)
@@ -35,5 +35,5 @@
 				</clip>
 			</camera>
-			<topic>camera/image_raw</topic>
+			<topic>$(arg namespace)/camera/image_raw</topic>
             <gz_frame_id>CAMERA_OPTICAL</gz_frame_id>
 		</sensor>
