Commit message: removed the pycache and made some changes to the jetank's camera

File: jetank_description/urdf/jetank_joints.xacro (robot description, xacro)
@@ -73,4 +73,10 @@
         <limit lower="0" upper="${PI/4}" effort="75" velocity="10" />
     </xacro:joint>
+    <!-- CAMERA -->
+    <xacro:joint joint_name="ARM_LOWER_rigid_CAMERA_HOLDER_ARM_LOWER" parent_name="ARM_LOWER" child_name="CAM_HOLDER" joint_type="revolute">
+        <origin xyz="-0.0248 0 0.0344" rpy="${PI/2} ${-PI/16} 0" />
+        <axis xyz="1 0 0"/>
+        <limit lower="0" upper="${PI/4}" effort="75" velocity="10"/>
+    </xacro:joint>
     <!-- fixed joints -->
     <xacro:joint joint_name="base_link_rigid_ANTENNA_L_BASE_JOINT" parent_name="base_link" child_name="ANTENNA_L" joint_type="fixed">
@@ -94,9 +100,4 @@
         <limit/>
     </xacro:joint>
-    <xacro:joint joint_name="ARM_LOWER_rigid_CAMERA_HOLDER_ARM_LOWER" parent_name="ARM_LOWER" child_name="CAM_HOLDER" joint_type="fixed">
-        <origin xyz="-0.0248 0 0.0344" rpy="${PI/2} 0 0" />
-        <axis/>
-        <limit/>
-    </xacro:joint>
     <xacro:joint joint_name="ARM_LOWER_Rigid_SERVO_LOWER_ARM_LOWER" parent_name="ARM_LOWER" child_name="SERVO_LOWER" joint_type="fixed">
         <origin xyz="0.0135 0.0200 0.0672" rpy="${PI/2} 0 0" />

File: jetank_description/urdf/jetank_sensors.xacro (robot description, xacro)
@@ -23,5 +23,5 @@
 			<camera>
 				<camera_info_topic>camera/camera_info</camera_info_topic>
-				<horizontal_fov>1.089</horizontal_fov>
+				<horizontal_fov>1.5</horizontal_fov>
 				<image>
 					<!-- (RED) 8 bits + (BLUE) 8 bits  + (GREEN) 8 bits -->

Commit message: added custom messages for communication with the server and added a server node besides that modified some URDF settings

File: jetank_description/urdf/jetank_joints.xacro (robot description, xacro)
@@ -74,5 +74,5 @@
     </xacro:joint>
     <!-- CAMERA -->
-    <xacro:joint joint_name="ARM_LOWER_rigid_CAMERA_HOLDER_ARM_LOWER" parent_name="ARM_LOWER" child_name="CAM_HOLDER" joint_type="revolute">
+    <xacro:joint joint_name="ARM_LOWER_rigid_CAMERA_HOLDER_ARM_LOWER" parent_name="ARM_LOWER" child_name="CAM_HOLDER" joint_type="fixed">
         <origin xyz="-0.0248 0 0.0344" rpy="${PI/2} ${-PI/16} 0" />
         <axis xyz="1 0 0"/>

File: jetank_description/urdf/jetank_links.xacro (robot description, xacro)
@@ -42,7 +42,7 @@
             <origin xyz="-0.0028864851424563968 0.0003605395998919554 0.03729152724217677"
                 rpy="0.0 0.0 0.0" />
-            <mass value="0.7639308708503839" />
-            <inertia ixx="0.00150205741988797" iyy="0.003532242168965159" izz="0.003808278739772123"
-                ixy="2.0200689378287296e-06" iyz="4.791503412361428e-06" ixz="5.068154904514763e-05" />
+            <mass value="${base_link_mass}" />
+            <inertia ixx="0" iyy="0" izz="0"
+                ixy="0" iyz="0" ixz="0" />
         </inertial>
     </xacro:links>
@@ -53,5 +53,5 @@
             <origin xyz="-0.022908278643665785 0.0006057553402017391 -0.01928712656788768"
                 rpy="0.0 -4.220565730941431e-35 -6.162975822039156e-33" />
-            <mass value="0.03565761396104929" />
+            <mass value="${ARM_UPPER_mass}" />
             <inertia ixx="1.5443417400841932e-05" iyy="2.3764463595438004e-05"
                 izz="1.3620194048359787e-05" ixy="3.625928097526083e-06"
@@ -64,5 +64,5 @@
             <origin xyz="-0.03358748266767387 0.03358762804395098 -5.157163600578385e-05"
                 rpy="0.0 2.407412430484311e-35 1.2161079430919492e-49" />
-            <mass value="0.06186397464920469" />
+            <mass value="${ARM_MIDDLE_mass}" />
             <inertia ixx="6.497179907917266e-05" iyy="6.497176903594811e-05"
                 izz="6.838533670855049e-05" ixy="3.117958759744717e-05" iyz="1.061073116136028e-07"
@@ -75,5 +75,5 @@
             <origin xyz="-0.01064722156754466 -5.485356628246008e-05 0.029442007866704572"
                 rpy="4.814824860968091e-35 -0.0 3.2073176521106348e-49" />
-            <mass value="0.1036438493797283" />
+            <mass value="${ARM_LOWER_mass}" />
             <inertia ixx="8.81458213535141e-05" iyy="7.950393953510494e-05"
                 izz="7.219884111762218e-05" ixy="4.6845951821403056e-08" iyz="2.258742793083176e-07"
@@ -87,5 +87,5 @@
             <origin xyz="6.909868758699923e-05 -5.0523203168468815e-05 -0.019021631303903268"
                 rpy="0.0 1.8570051196622238e-34 0.0" />
-            <mass value="0.10496982138298995" />
+            <mass value="${DRIVER_WHEEL_L_mass}" />
             <inertia ixx="2.2560499003626737e-05" iyy="2.251410282101856e-05"
                 izz="2.4612100281121576e-05" ixy="-5.694123753574936e-11"
@@ -98,5 +98,5 @@
             <origin xyz="-6.909654809962084e-05 -2.9269046357853768e-05 -0.019021673226760922"
                 rpy="0.0 -6.360951486702456e-35 0.0" />
-            <mass value="0.1049698213829899" />
+            <mass value="${DRIVER_WHEEL_R_mass}" />
             <inertia ixx="2.2560499004256008e-05" iyy="2.251400779881374e-05"
                 izz="2.4612195302702004e-05" ixy="-2.5324020125478572e-11"
@@ -109,5 +109,5 @@
             <origin xyz="4.913425615981737e-05 -2.8359849328207787e-05 -0.01352728007660148"
                 rpy="0.0 1.8570051196622238e-34 0.0" />
-            <mass value="0.11488889485414525" />
+            <mass value="${FREE_WHEEL_L_mass}" />
             <inertia ixx="4.0681765416765274e-05" iyy="4.068201157526234e-05"
                 izz="4.0263672111597786e-05" ixy="3.7418240329583945e-12"
@@ -120,5 +120,5 @@
             <origin xyz="-4.91456850747074e-05 -2.8363712536370045e-05 -0.013527277364732724"
                 rpy="0.0 -6.360951486702456e-35 0.0" />
-            <mass value="0.11488889485415185" />
+            <mass value="${FREE_WHEEL_R_mass}" />
             <inertia ixx="4.0681765245256105e-05" iyy="4.0682011546281835e-05"
                 izz="4.0263672312089414e-05" ixy="-3.654323655849692e-13"
@@ -132,5 +132,5 @@
             <origin xyz="-0.005467113295410968 -4.792118534928669e-06 0.0028147721817248163"
                 rpy="0.0 -0.0 -1.1739041031382518e-47" />
-            <mass value="0.019177097425958016" />
+            <mass value="${CAMERA_mass}" />
             <inertia ixx="1.2125641079973622e-06" iyy="1.0782087605613606e-06"
                 izz="9.171773161657565e-07" ixy="1.5309653202804099e-09"
@@ -143,5 +143,5 @@
             <origin xyz="-0.022309879542198107 1.7398627940234946e-06 -8.10411995800453e-05"
                 rpy="0.0 -2.0981802744010314e-34 -1.88079096131566e-37" />
-            <mass value="0.04320508566431304" />
+            <mass value="${CAMERA_HOLDER_mass}" />
             <inertia ixx="2.5816875300630775e-05" iyy="3.164288509735364e-05"
                 izz="1.2443592739336833e-05" ixy="7.560146391039103e-10"
@@ -155,5 +155,5 @@
             <origin xyz="-1.4377769774753802e-08 5.306325474567775e-06 -0.0025299943110332545"
                 rpy="0.0 -0.0 -8.784755544884209e-38" />
-            <mass value="0.05589211207057759" />
+            <mass value="${BEARING_mass}" />
             <inertia ixx="9.015512369875424e-06" iyy="9.015545628046614e-06"
                 izz="1.657627265380158e-05" ixy="-6.040612411177808e-14"
@@ -167,5 +167,5 @@
             <origin xyz="0.00010428589158372858 0.05125494812152533 -0.028760898470254075"
                 rpy="0.0 1.8570051196622238e-34 0.0" />
-            <mass value="0.1712590340150529" />
+            <mass value="${ANTENNA_L_mass}" />
             <inertia ixx="0.000314068362815308" iyy="1.1348965126681299e-05"
                 izz="0.0003064181988690546" ixy="-7.600553009246833e-08"
@@ -178,5 +178,5 @@
             <origin xyz="-0.00010388848222362413 -0.05137513349335263 -0.028545652272082785"
                 rpy="0.0 -6.360951486702456e-35 0.0" />
-            <mass value="0.17125903401505282" />
+            <mass value="${ANTENNA_R_mass}" />
             <inertia ixx="0.00031406836395675376" iyy="1.117596753400613e-05"
                 izz="0.00030659119532028506" ixy="-7.381378770492805e-08"
@@ -190,5 +190,5 @@
             <origin xyz="-0.008710205981769175 -0.0008931796940865167 -0.0032610178523219346"
                 rpy="0.0 -0.0 8.152758619563242e-34" />
-            <mass value="0.20982161326472018" />
+            <mass value="${SERVO_UPPER_mass}" />
             <inertia ixx="3.914539867865734e-05" iyy="3.5263719700624594e-05"
                 izz="5.518967950991577e-05" ixy="-3.681143850732295e-07"
@@ -201,5 +201,5 @@
             <origin xyz="-0.01778076329454675 -3.6698115345306094e-05 0.01751711641612725"
                 rpy="0.0 -0.0 5.473822126268817e-48" />
-            <mass value="0.20982161326471963" />
+            <mass value="${SERVO_LOWER_mass}" />
             <inertia ixx="3.6529219753117384e-05" iyy="5.780064634567519e-05"
                 izz="3.5268927790314385e-05" ixy="-1.2716158555447347e-09"
@@ -213,5 +213,5 @@
             <origin xyz="0.018711205204747332 0.007640083665599069 -0.007388532023619128"
                 rpy="0.0 -3.469446951953614e-18 -1.6155871338926322e-27" />
-            <mass value="0.0366550366587098" />
+            <mass value="${GRIPPER_BASE_mass}" />
             <inertia ixx="1.2285515330750476e-05" iyy="6.94612066955528e-06"
                 izz="1.715774480621983e-05" ixy="-9.121676749908667e-07"
@@ -224,5 +224,5 @@
             <origin xyz="-0.012998250088038078 -3.0306803820455697e-05 -0.008065030577021126"
                 rpy="0.0 -0.0 0.0" />
-            <mass value="0.0062442558314246485" />
+            <mass value="${GRIPPER_L1_mass}" />
             <inertia ixx="2.2945298088091447e-07" iyy="9.557086105196205e-07"
                 izz="7.526842531313375e-07" ixy="-2.161025306364326e-09"
@@ -235,5 +235,5 @@
             <origin xyz="-0.0012296239530053298 0.0039691186133053915 0.0036766615181430496"
                 rpy="0.0 -0.0 0.0" />
-            <mass value="0.02146027585992414" />
+            <mass value="${GRIPPER_L2_mass}" />
             <inertia ixx="1.2266606930363098e-06" iyy="6.125907172840806e-06"
                 izz="5.756214866640529e-06" ixy="-9.873904819377294e-07"
@@ -246,5 +246,5 @@
             <origin xyz="-0.012998246756733707 -3.0304779780740975e-05 -0.008065027151216597"
                 rpy="0.0 -0.0 0.0" />
-            <mass value="0.006244255831424673" />
+            <mass value="${GRIPPER_R1_mass}" />
             <inertia ixx="2.294529808805892e-07" iyy="9.557086105191868e-07"
                 izz="7.526842531311207e-07" ixy="-2.1610253063812667e-09"
@@ -257,5 +257,5 @@
             <origin xyz="-0.0012584873319152834 0.003975470401698931 -0.0036599972005064174"
                 rpy="0.0 -0.0 -6.018531076210082e-35" />
-            <mass value="0.021460275859939086" />
+            <mass value="${GRIPPER_R2_mass}" />
             <inertia ixx="1.2412063985862897e-06" iyy="6.1145027700224355e-06"
                 izz="5.753073563923234e-06" ixy="-1.0146443397531036e-06"

File: jetank_description/urdf/jetank_main.xacro (robot description, xacro)
@@ -53,5 +53,5 @@
     <xacro:property name="BEARING_material"                 value="0.67 0.74 0.67 1" />
     <!-- mass -->
-    <xacro:property name="base_link_mass"               value="2.7639308708503839" />
+    <xacro:property name="base_link_mass"               value="5.7639308708503839" />
     <xacro:property name="DRIVER_WHEEL_L_mass"          value="0.1049698213829899" />
     <xacro:property name="DRIVER_WHEEL_R_mass"          value="0.1049698213829899" />
@@ -105,8 +105,8 @@
     <xacro:property name="ARM_MIDDLE_dim"         value="${[0.115,  0.005,  0.05]}"/>
     <xacro:property name="ARM_LOWER_dim"          value="${[0.06,  0.02,  0.0]}"/>
-    <xacro:property name="DRIVER_WHEEL_L_dim"     value="${[0.025,  0.025,  0.0]}"/>
-    <xacro:property name="DRIVER_WHEEL_R_dim"     value="${[0.025,  0.025,  0.0]}"/>
-    <xacro:property name="FREE_WHEEL_L_dim"       value="${[0.025,  0.025,  0.0]}"/>
-    <xacro:property name="FREE_WHEEL_R_dim"       value="${[0.025,  0.025,  0.0]}"/>
+    <xacro:property name="DRIVER_WHEEL_L_dim"     value="${[0.03,  0.03,  0.0]}"/>
+    <xacro:property name="DRIVER_WHEEL_R_dim"     value="${[0.03,  0.03,  0.0]}"/>
+    <xacro:property name="FREE_WHEEL_L_dim"       value="${[0.03,  0.03,  0.0]}"/>
+    <xacro:property name="FREE_WHEEL_R_dim"       value="${[0.03,  0.03,  0.0]}"/>
     <xacro:property name="CAMERA_dim"             value="${[0.01,  0.01,  0.01]}"/>
     <xacro:property name="CAMERA_HOLDER_dim"      value="${[0.05,  0.02,  0]}"/>
